File: control_contactor_v2/control_contactor_v2.kicad_sch (KiCad schematic)
At the start: 0 parts

Commit message: react + v2.2
Parts:
- added 1Meg: 1Mohm, symbol Device:R
- added 5k: 5kohm, symbol Device:R
- added AIR+, AIR-, PRE-CHARGE: Relay_DPST-NO, symbol Relay:Relay_DPST-NO
- added C1: 100nf, symbol Device:C
- added C2, C3: 1nF, symbol Device:C
- added D1, D2, D4: D, symbol Device:D
- added Q1, Q2, Q3: Q_NMOS_GDS, symbol Transistor_FET:Q_NMOS_GDS
- added R1, R10, R11, R2, R3, R8, R9: 10k, symbol Device:R
- added R4: 100ohm_50w, symbol Device:R
- added R5, R6, R7: R, symbol Device:R
- added U1: ISO224xDWV, Package_SO:SOIC-8_7.5x5.85mm_P1.27mm, symbol Isolator_Analog:ISO224xDWV
- added U2: ${SIM.PARAMS}, symbol Simulation_SPICE:OPAMP
Connections:
- new net: AIR-.A2, D4.2 (A), Q2.2 (D)
- new net: D2.2 (A), PRE-CHARGE.A2, Q3.2 (D)
- new net: PRE-CHARGE.23, R4.1
- new net: C2.1, R10.2, R11.1, U2.2 (-)
- new net: C3.1, R8.2, R9.2, U2.1 (+)
- new net: AIR+.A2, D1.2 (A), Q1.2 (D)
- new net +24V: D2.1 (K), PRE-CHARGE.A1
- new net +24V SDC: AIR+.A1, AIR-.A1, D1.1 (K), D4.1 (K)
- new net +3.3V: AIR+.14, AIR-.14, PRE-CHARGE.14
- new net +5V: U1.8 (VDD2), U2.3 (V+)
- new net +5V_ISO: U1.3 (VDD1)
- new net CTRL_AIR_MINUS: Q2.1 (G), R2.1
- new net CTRL_AIR_PLUS: Q1.1 (G), R1.1
- new net CTRL_PRECHARGE: Q3.1 (G), R3.1
- new net FB_AIR_MINUS: PRE-CHARGE.13, R6.1
- new net FB_AIR_PLUS: AIR+.13, R5.1
- new net FB_PRECHARGE: AIR-.13, R7.1
- new net GND: C3.2, Q1.3 (S), Q2.3 (S), Q3.3 (S), R1.2, R2.2, R3.2, R5.2, R6.2, R7.2, R9.1, U1.5 (GND2), U2.4 (V-)
- new net HV_BAT+: AIR+.24, PRE-CHARGE.24
- new net HV_BAT-: AIR-.24
- new net HV_GND: 5k.2, C1.2, U1.1 (VCAP), U1.4 (GND1)
- new net HV_INV+: 1Meg.1, AIR+.23, R4.2
- new net HV_INV-: AIR-.23
- new net HV_SENSE_RAW: 1Meg.2, 5k.1, C1.1, U1.2 (IN)
- new net HV_SENSE_SAFE: C2.2, R11.2, U2.5
- new net ISO_OUT_N: R10.1, U1.6 (OUTN)
- new net ISO_OUT_P: R8.1, U1.7 (OUTP)
Other:
- note added: "Depends on the contactor: 1. C7- needed 2. Gigavac- not needed"

Commit message: v2 final
Parts:
- added C4: 100nf, symbol Device:C
- added R12: 1kohm, symbol Device:R
- added R13: 100kohm, symbol Device:R
- added R14: 10k, symbol Device:R
- added RV1: R_Potentiometer_Trim, symbol Device:R_Potentiometer_Trim
- added U3: LM393, symbol Comparator:LM393
Connections:
- net +5V: now also RV1.1, U3.8 (V+)
- net GND: now also C4.2, RV1.3, U3.4 (V-), U3.5 (+), U3.6 (-)
- net HV_SENSE_SAFE: now also R12.1
- new net: C4.1, RV1.2, U3.2 (-)
- new net: R12.2, R13.1, U3.3 (+)
- new net STM 3.3v rail: R14.1
- new net STM input: R13.2, R14.2, U3.1
Other:
- note added: "==================================================================== HV PRECHARGE SENSING & HARDWARE THRESHOLD CIRCUIT Overview: This circuit safely steps down, isolates, and monitors the High Voltage (HV) traction bus. It provides both a continuous analog telemetry signal and a hardware-level digital trigger to the MCU for executing the Make-Before-Break precharge contactor sequence. Stage 1: HV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"
- note added: "difference op-amp"
- note added: "isolation amplifier"
- moved on the sheet: 1Meg, 5k, AIR-, C1, C2, C3, D2, D4, PRE-CHARGE, Q2, Q3, R10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

Commit message: 12may isolation amplifier, transformer, etc
Parts:
- removed R10, R11, R14, R9: 10k, symbol Device:R
- removed R12: 1kohm, symbol Device:R
- removed R13: 100kohm, symbol Device:R
- removed U1: ISO224xDWV, Package_SO:SOIC-8_7.5x5.85mm_P1.27mm, symbol Isolator_Analog:ISO224xDWV
- removed U2: ${SIM.PARAMS}, symbol Simulation_SPICE:OPAMP
- removed U3: LM393, symbol Comparator:LM393
- added D3, D5: MBR0520LT, Diode_SMD:D_SOD-123, symbol Diode:MBR0520LT
- added TR1: Wuerth_750315371, Transformer_SMD:Transformer_Wuerth_750315371, symbol Transformer:Wuerth_750315371
- added U1: LM7805_TO220, Package_TO_SOT_THT:TO-220-3_Vertical, symbol Regulator_Linear:LM7805_TO220
- added U2: LM393, symbol Comparator:LM393
- added U3: AMC1301DWVR, DWV0008A, symbol 2026-05-11_16-05-38:AMC1301DWVR
- added U4: SN6501DBVR, DBV0005A_N, symbol 2026-05-12_02-25-53:SN6501DBVR
- added U5: TPS76350DBVR, DBV5, symbol 2026-05-12_02-50-01:TPS76350DBVR
- added r11, r12, r9: 200kΩ, symbol Device:R
- added r14: 1Mohm, symbol Device:R
- C2, C3: value 1nF -> 100nf
- R5, R6: value R -> 10kohm
- R7: value R -> 100ohm
- R8: value 10k -> 10kohm
- r10: renamed from 1Meg; value 1Mohm -> 200kΩ
- r13: renamed from 5k; value 5kohm -> 1kΩ
- renumbered AIR+ to AIR+1, AIR- to AIR-1, PRE-CHARGE to PRE-CHARGE1
Connections:
- net HV_SENSE_SAFE is gone; now on net GND: C2.2
- net ISO_OUT_P is gone; now on net 5v_comp: R8.1
- net +24V: now also C2.1, U1.1 (VI)
- net +3.3V: now also C4.1, TR1.2, U2.8 (V+), U3.8 (VDD2), U4.2 (VCC)
- net GND: now also C3.1, U1.2 (GND), U2.4 (V-), U2.5 (+), U2.6 (-), U3.5 (GND2), U4.4 (GND), U4.5 (GND); no longer C3.2
- net HV_INV+: now also r11.1; no longer r10.1
- net HV_SENSE_RAW: now also U3.2 (VINP)
- net vref_comp: now reaches RV1.2
- net vref_comp: now also U2.2 (-); no longer C4.1
- net stem_input: now reaches R8.2
- net stem_input: now also U2.1, r14.2; no longer C3.1
- net +5V renamed 5v_comp
- net 5v_comp: now also C3.2, U1.3 (VO)
- net HV_GND renamed GND2
- net GND2: now also TR1.5, U3.3 (VINN), U3.4 (GND1), U5.2 (GND)
- new net: D3.1 (K), D5.1 (K), U5.1 (IN), U5.3 (EN)
- new net: U3.1 (VDD1), U5.5 (OUT)
- new net: U2.3 (+), U3.7 (VOUTP), r14.1
- new net: TR1.1, U4.1 (D1)
- new net: TR1.3, U4.3 (D2)
- new net: D5.2 (A), TR1.4
- new net: D3.2 (A), TR1.6
- new net: r10.1, r9.2
- new net: r12.2, r9.1
- new net: r11.2, r12.1
Other:
- note added: "GND - lv GND2 - HV"
- note added: "set voltage to 3.48v"
- note removed: "==================================================================== HV PRECHARGE SENSING & HARDWARE THRESHOLD CIRCUIT Overview: This circuit safely steps down, isolates, and monitors the High Voltage (HV) traction bus. It provides both a continuous analog telemetry signal and a hardware-level digital trigger to the MCU for executing the Make-Before-Break precharge contactor sequence. Stage 1: HV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"
- note removed: "difference op-amp"
- note removed: "isolation amplifier"
- moved on the sheet: C1, r10, r13
